File: HE75.kicad_pcb (KiCad board)
At the start: 4 copper layers, 285 x 94.6 mm, 278 parts, among them J1 USB_C_Receptacle_USB2.0_16P, SW1 Esc, SW10 9, SW11 0, SW12 -, SW13 =, SW14 Bksp, SW15 Del, SW16 Tab, SW17 Q, SW18 W, SW19 E, SW2 1, SW20 R, SW21 T, SW22 Y, SW23 U, SW24 I, SW25 O, SW26 P, SW27 [, SW28 ], SW29 \, SW3 2, SW30 Pg Up, SW31 Caps, SW32 A, SW33 S, SW34 D, SW35 F, SW36 G, SW37 H, SW38 J, SW39 K, SW4 3, SW40 L, SW41 ;, SW42 ', SW43 Enter, SW44 End, SW45 Pg Dn, SW46 Shift, SW47 Z, SW48 X, SW49 C, SW5 4, SW50 V, SW51 B, SW52 N, SW53 M, SW54 ,, SW55 ., SW56 /, SW57 Shift, SW58 Home, SW59 Up, SW6 5, SW60 Code, SW61 Fn, SW62 Ctrl, SW63 Win, SW64 Alt, SW65 Space, SW66 Space, SW67 Space, SW68 Space, SW69 Alt, SW7 6, SW70 Win, SW71 Ctrl, SW72 Fn, SW73 Left, SW74 Down, SW75 Right, SW76 Space L2u, SW77 Space C2u, SW78 Space R2u, SW8 7, SW9 8, U1 STM32F303CCT6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

Commit message: Cleanup
Parts:
- removed the C10 at (71.4, 43.2)
- removed the C11 at (70.8, 41.8)
- removed FB2: 600R, Inductor_SMD:L_0805_2012Metric
- added C8: 1uF, Library:Capacitor 0402, B.Cu at (74.5, 50.3)
- added C9: 100nF, Library:Capacitor 0402, B.Cu at (75.5, 48.1)
- C2: value 10nF -> 4.7uF
- C3, C5: value 1uF -> 100nF
- C6: value 4.7uF -> 10nF
- C7: value 100nF -> 1uF
- F1: footprint Fuse:Fuse_1206_3216Metric -> Fuse:Fuse_0805_2012Metric
- J1: footprint Connector_USB:USB_C_Receptacle_HRO_TYPE-C-31-M-12 -> Library:USB_C_Receptacle_HRO_TYPE-C-31-M-12
- moved R1 26.9 mm to (47.8, 52.4), turned to 0 degrees
- moved C12 22.8 mm to (41.2, 46.1), turned to 90 degrees
- moved RST1 22.4 mm to (50.6, 48.9), turned to 180 degrees
- moved C13 20.0 mm to (44.8, 48.4)
- moved U2 19.9 mm to (44.2, 46.1)
- moved AM4 19.1 mm to (295.2, 86.2)
- moved AM0 19.1 mm to (66.7, 86.2)
- moved AM1 19.0 mm to (123.8, 86.2)
- moved AM2 19.0 mm to (180.9, 86.2)
- moved AM3 19.0 mm to (238.1, 86.2)
- moved F1 16.3 mm to (42.1, 42.6), turned to -90 degrees
- moved D1 13.8 mm to (44.0, 43.0), turned to -90 degrees
- moved C3 13.2 mm to (60.5, 43.5), turned to 90 degrees
- moved C11 11.6 mm to (74.4, 46.3), turned to -45 degrees
- moved C1 11.5 mm to (63.3, 51.9), turned to 180 degrees
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- renumbered U4 to AM0, U5 to AM1, U6 to AM2, U7 to AM3, U8 to AM4, C12 to C10, C13 to C11, C8 to C12, C9 to C13, U3 to U2
Connections:
- net /AM0 renamed /ADC4_IN3
- AM1 pad 1: /AM1 -> /ADC3_IN1
- AM2 pad 1: /AM2 -> /ADC3_IN12
- AM3 pad 1: /AM3 -> /ADC2_IN2
- AM4 pad 1: /AM4 -> /ADC2_IN1
- C1 pad 1: /NRST -> GND
- C1 pad 2: GND -> +3.3V
- C2 pad 2: +3.3VA -> +3.3V
- C3 pad 2: +3.3VA -> +3.3V
- C6 pad 2: +3.3V -> +3.3VA
- C7 pad 2: +3.3V -> +3.3VA
- H1 pad 1: GNDPWR -> (no net)
- HE1 pad 2: /A06 -> /A05
- HE10 pad 2: /A54 -> /A53
- HE11 pad 2: /A53 -> /A51
- HE13 pad 2: /A70 -> /A69
- HE14 pad 2: /A69 -> /A67
- HE16 pad 2: /A07 -> /A06
- HE19 pad 2: /A23 -> /A22
- HE2 pad 2: /A05 -> /A03
- HE22 pad 2: /A39 -> /A38
- HE25 pad 2: /A55 -> /A54
- HE28 pad 2: /A71 -> /A70
- HE32 pad 2: /A03 -> /A07
- HE35 pad 2: /A19 -> /A23
- HE38 pad 2: /A35 -> /A39
- HE4 pad 2: /A22 -> /A21
- HE40 pad 2: /A63 -> /A56
- HE41 pad 2: /A51 -> /A55
- HE44 pad 2: /A67 -> /A71
- HE47 pad 2: /A12 -> /A10
- HE5 pad 2: /A21 -> /A19
- HE50 pad 2: /A29 -> /A26
- HE53 pad 2: /A46 -> /A42
- HE54 pad 2: /A56 -> /A57
- HE55 pad 2: /A57 -> /A58
- HE56 pad 2: /A60 -> /A59
- HE57 pad 2: /A62 -> /A63
- HE59 pad 2: /A76 -> /A74
- HE61 pad 2: /A10 -> /A11
- HE62 pad 2: /A11 -> /A12
- HE64 pad 2: /A26 -> /A27
- HE67 pad 2: /A43 -> /A44
- HE68 pad 2: /A45 -> /A46
- HE7 pad 2: /A38 -> /A37
- HE70 pad 2: /A58 -> /A60
- HE71 pad 2: /A59 -> /A61
- HE72 pad 2: /A61 -> /A62
- HE73 pad 2: /A74 -> /A75
- HE74 pad 2: /A75 -> /A76
- HE76 pad 2: /A27 -> /A29
- HE77 pad 2: /A42 -> /A43
- HE78 pad 2: /A44 -> /A45
- HE8 pad 2: /A37 -> /A35
- J1 pad S1: GNDPWR -> GND
- U1 pad 12: /AM4 -> unconnected-(U1-PA2-Pad12)
- U1 pad 13: /AM3 -> unconnected-(U1-PA3-Pad13)
- U1 pad 14: unconnected-(U1-PA4-Pad14) -> /ADC2_IN1
- U1 pad 15: unconnected-(U1-PA5-Pad15) -> /ADC2_IN2
- U1 pad 16: /AM2 -> unconnected-(U1-PA6-Pad16)
- U1 pad 17: /AM1 -> unconnected-(U1-PA7-Pad17)
- U1 pad 18: unconnected-(U1-PB0-Pad18) -> /ADC3_IN12
- U1 pad 19: /S3 -> /ADC3_IN1
- U1 pad 20: /S2 -> unconnected-(U1-PB2-Pad20)
- U1 pad 21: /S1 -> unconnected-(U1-PB10-Pad21)
- U1 pad 22: /S0 -> unconnected-(U1-PB11-Pad22)
- U1 pad 40: unconnected-(U1-PB4-Pad40) -> /S3
- U1 pad 41: unconnected-(U1-PB5-Pad41) -> /S2
- U1 pad 42: unconnected-(U1-PB6-Pad42) -> /S0
- U1 pad 43: unconnected-(U1-PB7-Pad43) -> /S1
Routing:
- net GNDPWR: track 303.1 -> 0.00 mm
- net /S3: track 276.9 -> 528.6 mm, vias 8 -> 2
- net /S0: track 270.3 -> 512.5 mm, vias 2 -> 8
- net /ADC2_IN1: track 0.00 -> 240.1 mm, vias 0 -> 2
- net /S2: track 282.4 -> 520.8 mm, vias 4 -> 8
- net /S1: track 270.6 -> 498.8 mm, vias 6 -> 10
- net /AM4: track 215.5 -> 0.00 mm, vias 2 -> 0
- net /ADC2_IN2: track 0.00 -> 184.1 mm, vias 0 -> 2
- net /AM3: track 159.1 -> 0.00 mm, vias 2 -> 0
- net /ADC3_IN12: track 0.00 -> 128.5 mm, vias 0 -> 2
- net /AM2: track 103.9 -> 0.00 mm, vias 2 -> 0
- net /ADC3_IN1: track 0.00 -> 73.1 mm, vias 0 -> 2
- net GND: track 410.7 -> 346.8 mm, vias 109 -> 103
- net +3.3VA: track 280.8 -> 227.9 mm
- net /AM1: track 52.4 -> 0.00 mm, vias 2 -> 0
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
Commit message: Fix sot-143b footprint
Parts:
- C8, FB1: moved to F.Cu
- D2: footprint Package_TO_SOT_SMD:SOT-143 -> Library:SOT-143B
- moved C8 87.4 mm to (0.94, 3.23), turned to 0 degrees
- moved FB1 86.5 mm to (1.77, 0.88), turned to 0 degrees
- moved C12 62.7 mm to (17.0, -11.8)
- moved C4 62.7 mm to (44.9, -17.4)
- moved C5 62.7 mm to (47.6, -15.4)
- moved F1 62.7 mm to (18.0, -15.3)
- moved U2 62.7 mm to (20.1, -11.8)
- moved Y1 62.7 mm to (51.8, -13.1)
- moved C1 62.7 mm to (39.2, -6.01)
- moved C10 62.7 mm to (53.4, -14.7)
- moved C11 62.7 mm to (50.2, -11.6)
- moved C13 62.7 mm to (20.7, -9.50)
- moved C2 62.7 mm to (39.2, -5.01)
- moved C3 62.7 mm to (36.3, -14.4)
- moved C6 62.7 mm to (48.7, -9.32)
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Routing:
- net /S3: track 528.6 -> 0.00 mm, vias 2 -> 0
- net /S2: track 520.8 -> 0.00 mm, vias 8 -> 0
- net /S0: track 512.5 -> 0.00 mm, vias 8 -> 0
- net /S1: track 498.8 -> 0.00 mm, vias 10 -> 0
- net /ADC2_IN1: track 240.1 -> 0.00 mm, vias 2 -> 0
- net /ADC2_IN2: track 184.1 -> 0.00 mm, vias 2 -> 0
- net /ADC3_IN12: track 128.5 -> 0.00 mm, vias 2 -> 0
- net /ADC3_IN1: track 73.1 -> 0.00 mm, vias 2 -> 0
- net +3.3V: track 68.5 -> 0.00 mm, vias 2 -> 0
- net /ADC4_IN3: track 57.6 -> 0.00 mm, vias 4 -> 0
- net GND: track 346.8 -> 311.6 mm, vias 103 -> 93
- net /BOOT0: track 28.2 -> 0.00 mm, vias 4 -> 0
- net /USB_D+: track 26.9 -> 7.53 mm
- net /USB_D-: track 24.2 -> 7.53 mm
- net /CC1: track 13.1 -> 1.38 mm, vias 2 -> 1
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- added copper zone on In1.Cu, net +3.3VA
- removed copper zone on F.Cu, net +3.3VA
- removed copper zone on In1.Cu, net GND

Commit message: Fills
Parts:
- removed D2: PRTR5V0U2X, Library:SOT-143B
- removed FID (x3): FIDUCIAL, hole:FIDUCIAL
- removed HOLE (x2): VAL**, hole:PKRH
- removed HOLE: VAL**, hole:PKRHC
- removed HOLE (x2): VAL**, hole:PKRHSL
- added H2: MountingHole, MountingHole:MountingHole_2.2mm_M2, F.Cu at (250.6, 136.3)
- added H3: MountingHole, MountingHole:MountingHole_2.2mm_M2, F.Cu at (256.5, 130.4)
- added H4: MountingHole, MountingHole:MountingHole_2.2mm_M2, F.Cu at (256.5, 136.3)
- added H5: MountingHole, MountingHole:MountingHole_2.2mm_M2, F.Cu at (262.5, 130.4)
- added H6: MountingHole, MountingHole:MountingHole_2.2mm_M2, F.Cu at (262.5, 136.3)
- added H7: MountingHole, MountingHole:MountingHole_2.2mm_M2, F.Cu at (268.4, 130.4)
- added H8: MountingHole, MountingHole:MountingHole_2.2mm_M2, F.Cu at (268.4, 136.3)
- added O1: GH60 Outline, Library:60_Outline, F.Cu at (171.4, 76.2)
- added U3: XC6206PxxxMR, Package_TO_SOT_SMD:SOT-23-3, B.Cu at (44.2, 47.1)
- C8, FB1: moved to B.Cu
- H1: footprint Library:Grounding Hole -> MountingHole:MountingHole_2.2mm_M2
- U2: value XC6206PxxxMR -> TPD4E05U06DQAR; footprint Package_TO_SOT_SMD:SOT-23-3 -> Package_SON:USON-10_2.5x1.0mm_P0.5mm
- moved Y1 92.1 mm to (47.6, 78.8), turned to 180 degrees
- moved C10 91.4 mm to (48.3, 76.6), turned to 180 degrees
- moved C11 88.4 mm to (46.4, 76.7), turned to 0 degrees
- moved C5 85.9 mm to (49.9, 70.5)
- moved C4 84.8 mm to (52.5, 67.1), turned to -90 degrees
- moved C9 84.1 mm to (46.8, 74.1), turned to -90 degrees
- moved FB1 80.9 mm to (42.5, 70.8)
- moved C7 80.0 mm to (45.5, 71.4), turned to 180 degrees
- moved C6 79.6 mm to (45.5, 70.2), turned to 180 degrees
- moved C8 78.1 mm to (40.2, 70.8), turned to 90 degrees
- moved U1 76.4 mm to (46.7, 64.6), turned to 90 degrees
- moved C3 74.2 mm to (49.3, 58.7), turned to 0 degrees
- moved R4 71.9 mm to (48.5, 56.1), turned to 0 degrees
- moved C1 68.2 mm to (40.8, 62.1), turned to 90 degrees
- moved C2 67.2 mm to (39.6, 62.1), turned to 90 degrees
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Connections:
- U1 pad 40: /S3 -> /S0
- U1 pad 41: /S2 -> /S1
- U1 pad 42: /S0 -> /S3
- U1 pad 43: /S1 -> /S2
- U2 pad 1: GND -> /USB_D+
- U2 pad 2: +3.3V -> /USB_D+
- U2 pad 3: +5V -> GND
Routing:
- net /S3: track 0.00 -> 258.6 mm, vias 0 -> 5
- net /S0: track 0.00 -> 258.5 mm, vias 0 -> 6
- net /S2: track 0.00 -> 258.3 mm, vias 0 -> 5
- net /S1: track 0.00 -> 257.1 mm, vias 0 -> 6
- net /A69: track 55.1 -> 0.00 mm
- net /A53: track 55.1 -> 0.00 mm
- net /A37: track 55.1 -> 0.00 mm
- net /A21: track 55.1 -> 0.00 mm
- net /A05: track 55.1 -> 0.00 mm
- net /A43: track 52.6 -> 0.00 mm
- net /A19: track 48.9 -> 0.00 mm
- net /A67: track 48.9 -> 0.00 mm
- net /A51: track 48.9 -> 0.00 mm
- net /A35: track 48.9 -> 0.00 mm
- net /A03: track 48.9 -> 0.00 mm
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- added copper zone on B.Cu, net +3.3V
- added copper zone on F.Cu, net +3.3V
- added copper zone on B.Cu, net +3.3VA
- added copper zone on B.Cu, net GND
Other:
- outline, holes or cut-outs redrawn
- board text removed: "JLCJLCJLCJLC"

Commit message: Before attempting MCU rotation
Parts:
- moved RST1 25.6 mm to (37.7, 67.5), turned to 90 degrees
- moved R1 17.2 mm to (35.9, 62.6)
- moved VR13 5.02 mm to (264.4, 39.1), turned to 90 degrees
- moved VR14 5.02 mm to (283.4, 39.1), turned to 90 degrees
- moved VR15 5.02 mm to (302.5, 39.1), turned to 90 degrees
- moved VR24 5.02 mm to (188.2, 58.1), turned to 90 degrees
- moved VR28 5.02 mm to (264.4, 58.1), turned to 90 degrees
- moved VR30 5.02 mm to (302.5, 58.1), turned to 90 degrees
- moved VR39 5.02 mm to (188.2, 77.2), turned to 90 degrees
- moved VR43 5.02 mm to (264.4, 77.2), turned to 90 degrees
- moved VR44 5.02 mm to (283.4, 77.2), turned to 90 degrees
- moved VR45 5.02 mm to (302.5, 77.2), turned to 90 degrees
- moved VR54 5.02 mm to (188.2, 96.2), turned to 90 degrees
- moved VR58 5.02 mm to (264.4, 96.2), turned to 90 degrees
- moved VR59 5.02 mm to (283.4, 96.2), turned to 90 degrees
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Connections:
- HE16 pad 2: /A06 -> /A04
- HE17 pad 2: /A04 -> /A07
- HE19 pad 2: /A22 -> /A20
- HE20 pad 2: /A20 -> /A23
- HE22 pad 2: /A38 -> /A36
- HE23 pad 2: /A36 -> /A39
- HE25 pad 2: /A54 -> /A52
- HE26 pad 2: /A52 -> /A55
- HE29 pad 2: /A68 -> /A71
- HE31 pad 2: /A08 -> /A06
- HE32 pad 2: /A07 -> /A08
- HE34 pad 2: /A24 -> /A22
- HE35 pad 2: /A23 -> /A24
- HE37 pad 2: /A40 -> /A38
- HE38 pad 2: /A39 -> /A40
- HE40 pad 2: /A56 -> /A54
- HE41 pad 2: /A55 -> /A56
- HE43 pad 2: /A72 -> /A68
- HE44 pad 2: /A71 -> /A72
- HE48 pad 2: /A14 -> /A13
- HE51 pad 2: /A31 -> /A29
- HE54 pad 2: /A57 -> /A45
- HE55 pad 2: /A58 -> /A57
- HE56 pad 2: /A59 -> /A58
- HE57 pad 2: /A63 -> /A61
- HE60 pad 2: /A78 -> /A77
- HE63 pad 2: /A13 -> /A14
- HE66 pad 2: /A30 -> /A31
- HE67 pad 2: /A44 -> /A43
- HE68 pad 2: /A46 -> /A44
- HE69 pad 2: /A47 -> /A46
- HE70 pad 2: /A60 -> /A59
- HE71 pad 2: /A61 -> /A60
- HE75 pad 2: /A77 -> /A78
- HE76 pad 2: /A29 -> /A30
- HE77 pad 2: /A43 -> /A47
- HE78 pad 2: /A45 -> /A63
Routing:
- net /S3: track 258.6 -> 0.00 mm, vias 5 -> 0
- net /S0: track 258.5 -> 0.00 mm, vias 6 -> 0
- net /S2: track 258.3 -> 0.00 mm, vias 5 -> 0
- net /S1: track 257.1 -> 0.00 mm, vias 6 -> 0
- net /A63: track 0.00 -> 95.7 mm
- net /A47: track 0.00 -> 61.9 mm
- net /A59: track 0.00 -> 57.0 mm, vias 0 -> 3
- net /A43: track 0.00 -> 57.0 mm, vias 0 -> 3
- net /A27: track 0.00 -> 57.0 mm, vias 0 -> 3
- net /A11: track 0.00 -> 57.0 mm, vias 0 -> 3
- net /A04: track 0.00 -> 51.8 mm, vias 0 -> 2
- net /A31: track 0.00 -> 47.4 mm, vias 0 -> 1
- net /A62: track 0.00 -> 47.0 mm, vias 0 -> 2
- net /A46: track 0.00 -> 47.0 mm, vias 0 -> 2
- net /A14: track 0.00 -> 47.0 mm, vias 0 -> 2
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