File: HE75.kicad_pcb (KiCad board)
At the start: 4 copper layers, 285 x 94.6 mm, 277 parts, among them J1 USB_C_Receptacle_USB2.0_16P, SW1 Esc, SW10 9, SW11 0, SW12 -, SW13 =, SW14 Bksp, SW15 Del, SW16 Tab, SW17 Q, SW18 W, SW19 E, SW2 1, SW20 R, SW21 T, SW22 Y, SW23 U, SW24 I, SW25 O, SW26 P, SW27 [, SW28 ], SW29 \, SW3 2, SW30 Pg Up, SW31 Caps, SW32 A, SW33 S, SW34 D, SW35 F, SW36 G, SW37 H, SW38 J, SW39 K, SW4 3, SW40 L, SW41 ;, SW42 ', SW43 Enter, SW44 End, SW45 Pg Dn, SW46 Shift, SW47 Z, SW48 X, SW49 C, SW5 4, SW50 V, SW51 B, SW52 N, SW53 M, SW54 ,, SW55 ., SW56 /, SW57 Shift, SW58 Home, SW59 Up, SW6 5, SW60 Code, SW61 Fn, SW62 Ctrl, SW63 Win, SW64 Alt, SW65 Space, SW66 Space, SW67 Space, SW68 Space, SW69 Alt, SW7 6, SW70 Win, SW71 Ctrl, SW72 Fn, SW73 Left, SW74 Down, SW75 Right, SW76 Space L2u, SW77 Space C2u, SW78 Space R2u, SW8 7, SW9 8, U1 STM32F303CCT6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

Commit message: Complete
Parts:
- moved RST1 22.0 mm to (47.6, 47.9), turned to 180 degrees
- moved AM0 19.0 mm to (66.7, 85.8)
- moved AM1 19.0 mm to (123.9, 85.8)
- moved AM2 19.0 mm to (181.0, 85.8)
- moved AM3 19.0 mm to (238.2, 85.8)
- moved AM4 19.0 mm to (295.3, 85.8)
- moved R1 13.9 mm to (44.2, 51.5)
- moved U3 7.09 mm to (37.8, 50.0), turned to 180 degrees
- moved C13 5.93 mm to (38.2, 52.2), turned to 0 degrees
- moved C12 5.26 mm to (37.2, 47.8), turned to 180 degrees
- moved D1 3.56 mm to (40.0, 44.0)
- moved F1 2.01 mm to (37.8, 46.2), turned to 180 degrees
- moved C8 0.76 mm to (41.5, 72.8), turned to 90 degrees
- moved C9 0.11 mm to (46.2, 74.1)
Connections:
- AM0 pad 1: /ADC4_IN3 -> /ADC2_IN1
- AM1 pad 1: /ADC3_IN1 -> /ADC2_IN2
- AM3 pad 1: /ADC2_IN2 -> /ADC3_IN1
- AM4 pad 1: /ADC2_IN1 -> /ADC4_IN3
- HE1 pad 2: /A05 -> /A04
- HE10 pad 2: /A53 -> /A52
- HE12 pad 2: /A50 -> /A48
- HE13 pad 2: /A69 -> /A68
- HE15 pad 2: /A66 -> /A64
- HE16 pad 2: /A04 -> /A08
- HE17 pad 2: /A07 -> /A05
- HE19 pad 2: /A20 -> /A23
- HE20 pad 2: /A23 -> /A21
- HE22 pad 2: /A36 -> /A39
- HE23 pad 2: /A39 -> /A37
- HE25 pad 2: /A52 -> /A55
- HE26 pad 2: /A55 -> /A53
- HE28 pad 2: /A70 -> /A71
- HE29 pad 2: /A71 -> /A69
- HE3 pad 2: /A02 -> /A00
- HE32 pad 2: /A08 -> /A07
- HE33 pad 2: /A00 -> /A02
- HE34 pad 2: /A22 -> /A24
- HE35 pad 2: /A24 -> /A22
- HE36 pad 2: /A16 -> /A18
- HE37 pad 2: /A38 -> /A40
- HE38 pad 2: /A40 -> /A38
- HE39 pad 2: /A32 -> /A34
- HE4 pad 2: /A21 -> /A20
- HE40 pad 2: /A54 -> /A56
- HE41 pad 2: /A56 -> /A54
- HE42 pad 2: /A48 -> /A50
- HE43 pad 2: /A68 -> /A72
- HE44 pad 2: /A72 -> /A70
- HE45 pad 2: /A64 -> /A66
- HE46 pad 2: /A09 -> /A10
- HE47 pad 2: /A10 -> /A11
- HE48 pad 2: /A13 -> /A14
- HE49 pad 2: /A25 -> /A26
- HE50 pad 2: /A26 -> /A27
- HE51 pad 2: /A29 -> /A30
- HE53 pad 2: /A42 -> /A43
- HE54 pad 2: /A45 -> /A46
- HE55 pad 2: /A57 -> /A58
- HE56 pad 2: /A58 -> /A59
- HE57 pad 2: /A61 -> /A62
- HE58 pad 2: /A73 -> /A74
- HE59 pad 2: /A74 -> /A75
- HE6 pad 2: /A18 -> /A16
- HE60 pad 2: /A77 -> /A78
- HE61 pad 2: /A11 -> /A09
- HE63 pad 2: /A14 -> /A13
- HE64 pad 2: /A27 -> /A25
- HE67 pad 2: /A43 -> /A44
- HE68 pad 2: /A44 -> /A47
- HE69 pad 2: /A46 -> /A57
- HE7 pad 2: /A37 -> /A36
- HE70 pad 2: /A59 -> /A60
- HE71 pad 2: /A60 -> /A61
- HE72 pad 2: /A62 -> /A63
- HE73 pad 2: /A75 -> /A73
- HE75 pad 2: /A78 -> /A77
- HE76 pad 2: /A30 -> /A29
- HE77 pad 2: /A47 -> /A42
- HE78 pad 2: /A63 -> /A45
- HE9 pad 2: /A34 -> /A32
Routing:
- net /S0: track 0.00 -> 283.3 mm
- net /S1: track 0.00 -> 283.3 mm
- net /S2: track 0.00 -> 282.6 mm
- net /S3: track 0.00 -> 280.5 mm
- net /ADC4_IN3: track 21.4 -> 265.6 mm, vias 0 -> 2
- net /ADC3_IN1: track 0.00 -> 200.2 mm, vias 0 -> 2
- net /ADC3_IN12: track 0.00 -> 142.2 mm, vias 0 -> 2
- net /ADC2_IN2: track 0.00 -> 84.3 mm, vias 0 -> 2
- net /A63: track 95.7 -> 27.4 mm, vias 0 -> 2
- net /A08: track 8.36 -> 63.3 mm, vias 0 -> 2
- net /A75: track 57.0 -> 10.6 mm, vias 3 -> 2
- net /A59: track 57.0 -> 10.6 mm, vias 3 -> 2
- net /A43: track 57.0 -> 10.6 mm, vias 3 -> 2
- net /A27: track 57.0 -> 10.6 mm, vias 3 -> 2
- net /A11: track 57.0 -> 10.6 mm, vias 3 -> 2
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- added copper zone on B.Cu, net +5V
- removed copper zone on F.Cu, net +3.3V

Commit message: Add 6u spacebar stabalizers
Parts:
- added Stab4: MX_stab, PCM_marbastlib-mx:STAB_MX_6u, F.Cu at (142.9, 114.3)
- SW44: value End -> Home
- SW45: value Pg Dn -> End
- SW58: value Home -> Code
- SW60: value Code -> Pg Dn
- turned SW70 to 90 degrees
- turned SW71 to -90 degrees
Routing:
- net +3.3VA: track 236.4 -> 234.7 mm
- net /BOOT0: track 20.5 -> 19.0 mm

Commit message: Adjusting tracks and silkscreens
Parts:
- SW76: value Space L2u -> L2U
- SW77: value Space C2u -> C2U/6U
- SW78: value Space R2u -> R2U
- moved R1 6.74 mm to (51.0, 51.5)
- moved C8 2.26 mm to (43.2, 74.2), turned to 0 degrees
- moved FB1 1.59 mm to (43.7, 71.8), turned to 90 degrees
- renumbered RST1 to BOOT0
Routing:
- net /ADC4_IN3: track 265.6 -> 257.3 mm
- net /S1: track 283.3 -> 284.3 mm
- net /ADC3_IN1: track 200.2 -> 199.5 mm
- net /ADC2_IN1: track 33.4 -> 32.8 mm
- net +3.3VA: vias 95 -> 92
