File: HE75.kicad_pcb (KiCad board)
At the start: 4 copper layers, 285 x 94.6 mm, 278 parts, among them J1 USB_C_Receptacle_USB2.0_16P, SW1 Esc, SW10 9, SW11 0, SW12 -, SW13 =, SW14 Bksp, SW15 Del, SW16 Tab, SW17 Q, SW18 W, SW19 E, SW2 1, SW20 R, SW21 T, SW22 Y, SW23 U, SW24 I, SW25 O, SW26 P, SW27 [, SW28 ], SW29 \, SW3 2, SW30 Pg Up, SW31 Caps, SW32 A, SW33 S, SW34 D, SW35 F, SW36 G, SW37 H, SW38 J, SW39 K, SW4 3, SW40 L, SW41 ;, SW42 ', SW43 Enter, SW44 Home, SW45 End, SW46 Shift, SW47 Z, SW48 X, SW49 C, SW5 4, SW50 V, SW51 B, SW52 N, SW53 M, SW54 ,, SW55 ., SW56 /, SW57 Shift, SW58 Code, SW59 Up, SW6 5, SW60 Pg Dn, SW61 Fn, SW62 Ctrl, SW63 Win, SW64 Alt, SW65 Space, SW66 Space, SW67 Space, SW68 Space, SW69 Alt, SW7 6, SW70 Win, SW71 Ctrl, SW72 Fn, SW73 Left, SW74 Down, SW75 Right, SW76 L2U, SW77 C2U/6U, SW78 R2U, SW8 7, SW9 8, U1 STM32F303CCT6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

Commit message: Fixes for JLCPCB
Parts:
- Stab1: value MX_stab -> Left 2u; footprint PCM_marbastlib-mx:STAB_MX_2u -> Library:STAB_MX_2u
- Stab2: value MX_stab -> Center 2u; footprint PCM_marbastlib-mx:STAB_MX_2u -> Library:STAB_MX_2u
- Stab3: value MX_stab -> Right 2u; footprint PCM_marbastlib-mx:STAB_MX_2u -> Library:STAB_MX_2u
- Stab4: value MX_stab -> Center 6u; footprint PCM_marbastlib-mx:STAB_MX_6u -> Library:STAB_MX_6u
- moved H1 184.5 mm to (85.8, 47.5)
- moved H5 178.6 mm to (85.8, 104.7)
- moved H2 139.6 mm to (142.9, 47.5)
- moved H6 123.7 mm to (142.9, 104.7)
- moved H3 100.3 mm to (200.1, 47.5)
- moved H4 88.8 mm to (257.2, 47.5)
- moved H7 73.0 mm to (200.1, 104.7)
- moved H8 33.6 mm to (257.2, 104.7)
- moved C8 6.08 mm to (37.9, 71.2), turned to -90 degrees
- moved FB1 3.60 mm to (40.1, 71.2), turned to 0 degrees
- turned HE1 to 90 degrees
- turned HE10 to 90 degrees
- turned HE11 to 90 degrees
- turned HE12 to 90 degrees
- turned HE13 to 90 degrees
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Connections:
- U2 pad 1: /USB_D+ -> unconnected-(U2-D1+-Pad1)
- U2 pad 5: /USB_D- -> unconnected-(U2-D2--Pad5)
Routing:
- net +3.3V: track 21.2 -> 26.6 mm
- net +3.3VA: track 234.7 -> 231.4 mm
