File: HE75.kicad_sch (KiCad schematic)
At the start: 270 parts, among them J1 USB_C_Receptacle_USB2.0_16P, SW1 Esc, SW10 9, SW11 0, SW12 -, SW13 =, SW14 Bksp, SW15 Del, SW16 Tab, SW17 Q, SW18 W, SW19 E, SW2 1, SW20 R, SW21 T, SW22 Y, SW23 U, SW24 I, SW25 O, SW26 P, SW27 [, SW28 ], SW29 \, SW3 2, SW30 Pg Up, SW31 Caps, SW32 A, SW33 S, SW34 D, SW35 F, SW36 G, SW37 H, SW38 J, SW39 K, SW4 3, SW40 L, SW41 ;, SW42 ', SW43 Enter, SW44 End, SW45 Pg Dn, SW46 Shift, SW47 Z, SW48 X, SW49 C, SW5 4, SW50 V, SW51 B, SW52 N, SW53 M, SW54 ,, SW55 ., SW56 /, SW57 Shift, SW58 Home, SW59 Up, SW6 5, SW60 Code, SW61 Fn, SW62 Ctrl, SW63 Win, SW64 Alt, SW65 Space, SW66 Space, SW67 Space, SW68 Space, SW69 Alt, SW7 6, SW70 Win, SW71 Ctrl, SW72 Fn, SW73 Left, SW74 Down, SW75 Right, SW76 Space L2u, SW77 Space C2u, SW78 Space R2u, SW8 7, SW9 8, U1 STM32F303CCT6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

Commit message: Cleanup
Parts:
- removed C1: 100nF, Library:Capacitor 0402, symbol Device:C_Small
- removed FB2: 600R, Inductor_SMD:L_0805_2012Metric, symbol Device:FerriteBead
- removed H1: MountingHole, Library:Grounding Hole, symbol Mechanical:MountingHole_Pad
- added C9: 100nF, Library:Capacitor 0402, symbol Device:C_Small
- J1: footprint Connector_USB:USB_C_Receptacle_HRO_TYPE-C-31-M-12 -> Library:USB_C_Receptacle_HRO_TYPE-C-31-M-12
- Stab1, Stab2, Stab3: now left out of the parts list
- renumbered U4 to AM0, U5 to AM1, U6 to AM2, U7 to AM3, U8 to AM4, C7 to C1, C12 to C10, C13 to C11, C8 to C12, C9 to C13, C6 to C2, C4 to C3, C11 to C4, C10 to C5, C2 to C6, C3 to C7, C5 to C8, U3 to U2
Connections:
- net GNDPWR is gone; now on net GND: J1.S1 (SHIELD)
- net A03: now also HE2.2 (OUTPUT); no longer HE32.2 (OUTPUT)
- net A05: now also HE1.2 (OUTPUT); no longer HE2.2 (OUTPUT)
- net A06: now also HE16.2 (OUTPUT); no longer HE1.2 (OUTPUT)
- net A07: now also HE32.2 (OUTPUT); no longer HE16.2 (OUTPUT)
- net A10: now also HE47.2 (OUTPUT); no longer HE61.2 (OUTPUT)
- net A11: now also HE61.2 (OUTPUT); no longer HE62.2 (OUTPUT)
- net A12: now also HE62.2 (OUTPUT); no longer HE47.2 (OUTPUT)
- net A19: now also HE5.2 (OUTPUT); no longer HE35.2 (OUTPUT)
- net A21: now also HE4.2 (OUTPUT); no longer HE5.2 (OUTPUT)
- net A22: now also HE19.2 (OUTPUT); no longer HE4.2 (OUTPUT)
- net A23: now also HE35.2 (OUTPUT); no longer HE19.2 (OUTPUT)
- net A26: now also HE50.2 (OUTPUT); no longer HE64.2 (OUTPUT)
- net A27: now also HE64.2 (OUTPUT); no longer HE76.2 (OUTPUT)
- net A29: now also HE76.2 (OUTPUT); no longer HE50.2 (OUTPUT)
- net A35: now also HE8.2 (OUTPUT); no longer HE38.2 (OUTPUT)
- net A37: now also HE7.2 (OUTPUT); no longer HE8.2 (OUTPUT)
- net A38: now also HE22.2 (OUTPUT); no longer HE7.2 (OUTPUT)
- net A39: now also HE38.2 (OUTPUT); no longer HE22.2 (OUTPUT)
- net A42: now also HE53.2 (OUTPUT); no longer HE77.2 (OUTPUT)
- net A43: now also HE77.2 (OUTPUT); no longer HE67.2 (OUTPUT)
- net A44: now also HE67.2 (OUTPUT); no longer HE78.2 (OUTPUT)
- net A45: now also HE78.2 (OUTPUT); no longer HE68.2 (OUTPUT)
- net A46: now also HE68.2 (OUTPUT); no longer HE53.2 (OUTPUT)
- net A51: now also HE11.2 (OUTPUT); no longer HE41.2 (OUTPUT)
- net A53: now also HE10.2 (OUTPUT); no longer HE11.2 (OUTPUT)
- net A54: now also HE25.2 (OUTPUT); no longer HE10.2 (OUTPUT)
- net A55: now also HE41.2 (OUTPUT); no longer HE25.2 (OUTPUT)
- net A56: now also HE40.2 (OUTPUT); no longer HE54.2 (OUTPUT)
- net A57: now also HE54.2 (OUTPUT); no longer HE55.2 (OUTPUT)
- net A58: now also HE55.2 (OUTPUT); no longer HE70.2 (OUTPUT)
- net A59: now also HE56.2 (OUTPUT); no longer HE71.2 (OUTPUT)
- net A60: now also HE70.2 (OUTPUT); no longer HE56.2 (OUTPUT)
- net A61: now also HE71.2 (OUTPUT); no longer HE72.2 (OUTPUT)
- net A62: now also HE72.2 (OUTPUT); no longer HE57.2 (OUTPUT)
- net A63: now also HE57.2 (OUTPUT); no longer HE40.2 (OUTPUT)
- net A67: now also HE14.2 (OUTPUT); no longer HE44.2 (OUTPUT)
- net A69: now also HE13.2 (OUTPUT); no longer HE14.2 (OUTPUT)
- net A70: now also HE28.2 (OUTPUT); no longer HE13.2 (OUTPUT)
- net A71: now also HE44.2 (OUTPUT); no longer HE28.2 (OUTPUT)
- net A74: now also HE59.2 (OUTPUT); no longer HE73.2 (OUTPUT)
- net A75: now also HE73.2 (OUTPUT); no longer HE74.2 (OUTPUT)
- net A76: now also HE74.2 (OUTPUT); no longer HE59.2 (OUTPUT)
- net GND: now also C9.2
- net NRST: now also C9.1
- net S0: now also U1.42 (PB6); no longer U1.22 (PB11)
- net S1: now also U1.43 (PB7); no longer U1.21 (PB10)
- net S2: now also U1.41 (PB5); no longer U1.20 (PB2)
- net S3: now also U1.40 (PB4); no longer U1.19 (PB1)
- net ADC2_IN1: now reaches U1.14 (PA4)
- net ADC2_IN1: now also AM4.1 (COM)
- net ADC2_IN2: now reaches U1.15 (PA5)
- net ADC2_IN2: now also AM3.1 (COM)
- net ADC3_IN12: now reaches U1.18 (PB0)
- net ADC3_IN12: now also AM2.1 (COM)
- net AM0 renamed ADC4_IN3
- net AM1: no longer names the net of U1.17 (PA7)
- net AM1: no longer AM1.1 (COM)
- net AM2: no longer names the net of U1.16 (PA6)
- net AM2: no longer AM2.1 (COM)
- net AM3: no longer names the net of U1.13 (PA3)
- net AM3: no longer AM3.1 (COM)
- net AM4: no longer names the net of U1.12 (PA2)
- net AM4: no longer AM4.1 (COM)
- new net ADC3_IN1: AM1.1 (COM), U1.19 (PB1)
Other:
- note added: "Reset Pulldown"
- moved on the sheet: C10, C11, C2, C6, C7, C8, FB1, R1, R4, RST1, U1, Y1

Commit message: Fix sot-143b footprint
Parts:
- D2: footprint Package_TO_SOT_SMD:SOT-143 -> Library:SOT-143B
Changed lines of the file:
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@@
 			)
 		)
-		(property "Footprint" "Package_TO_SOT_SMD:SOT-143"
+		(property "Footprint" "Library:SOT-143B"
 			(at 196.85 71.374 0)
 			(effects

Commit message: Fills
Parts:
- removed D2: PRTR5V0U2X, Library:SOT-143B, symbol Power_Protection:PRTR5V0U2X
- added H1, H2, H3, H4, H5, H6, H7, H8: MountingHole, MountingHole:MountingHole_2.2mm_M2, symbol Mechanical:MountingHole
- added O1: GH60 Outline, Library:60_Outline, symbol Mechanical:Housing_Pad
- added U2: TPD4E05U06DQAR, Package_SON:USON-10_2.5x1.0mm_P0.5mm, symbol Power_Protection:TPD4E05U06DQA
- renumbered U2 to U3
Connections:
- net GND: now also O1.1 (PAD), U2.3 (GND), U2.8 (GND)
- net S0: now also U1.40 (PB4); no longer U1.42 (PB6)
- net S1: now also U1.41 (PB5); no longer U1.43 (PB7)
- net S2: now also U1.43 (PB7); no longer U1.41 (PB5)
- net S3: now also U1.42 (PB6); no longer U1.40 (PB4)
- net USB_D+: now also U2.1 (D1+), U2.2 (D1-), U2.9 (NC)
- net USB_D-: now also U2.4 (D2+), U2.5 (D2-), U2.7 (NC)
Other:
- moved on the sheet: D1, F1

Commit message: Before attempting MCU rotation
Connections:
- net A04: now also HE16.2 (OUTPUT); no longer HE17.2 (OUTPUT)
- net A06: now also HE31.2 (OUTPUT); no longer HE16.2 (OUTPUT)
- net A07: now also HE17.2 (OUTPUT); no longer HE32.2 (OUTPUT)
- net A08: now also HE32.2 (OUTPUT); no longer HE31.2 (OUTPUT)
- net A13: now also HE48.2 (OUTPUT); no longer HE63.2 (OUTPUT)
- net A14: now also HE63.2 (OUTPUT); no longer HE48.2 (OUTPUT)
- net A20: now also HE19.2 (OUTPUT); no longer HE20.2 (OUTPUT)
- net A22: now also HE34.2 (OUTPUT); no longer HE19.2 (OUTPUT)
- net A23: now also HE20.2 (OUTPUT); no longer HE35.2 (OUTPUT)
- net A24: now also HE35.2 (OUTPUT); no longer HE34.2 (OUTPUT)
- net A29: now also HE51.2 (OUTPUT); no longer HE76.2 (OUTPUT)
- net A30: now also HE76.2 (OUTPUT); no longer HE66.2 (OUTPUT)
- net A31: now also HE66.2 (OUTPUT); no longer HE51.2 (OUTPUT)
- net A36: now also HE22.2 (OUTPUT); no longer HE23.2 (OUTPUT)
- net A38: now also HE37.2 (OUTPUT); no longer HE22.2 (OUTPUT)
- net A39: now also HE23.2 (OUTPUT); no longer HE38.2 (OUTPUT)
- net A40: now also HE38.2 (OUTPUT); no longer HE37.2 (OUTPUT)
- net A43: now also HE67.2 (OUTPUT); no longer HE77.2 (OUTPUT)
- net A44: now also HE68.2 (OUTPUT); no longer HE67.2 (OUTPUT)
- net A45: now also HE54.2 (OUTPUT); no longer HE78.2 (OUTPUT)
- net A46: now also HE69.2 (OUTPUT); no longer HE68.2 (OUTPUT)
- net A47: now also HE77.2 (OUTPUT); no longer HE69.2 (OUTPUT)
- net A52: now also HE25.2 (OUTPUT); no longer HE26.2 (OUTPUT)
- net A54: now also HE40.2 (OUTPUT); no longer HE25.2 (OUTPUT)
- net A55: now also HE26.2 (OUTPUT); no longer HE41.2 (OUTPUT)
- net A56: now also HE41.2 (OUTPUT); no longer HE40.2 (OUTPUT)
- net A57: now also HE55.2 (OUTPUT); no longer HE54.2 (OUTPUT)
- net A58: now also HE56.2 (OUTPUT); no longer HE55.2 (OUTPUT)
- net A59: now also HE70.2 (OUTPUT); no longer HE56.2 (OUTPUT)
- net A60: now also HE71.2 (OUTPUT); no longer HE70.2 (OUTPUT)
- net A61: now also HE57.2 (OUTPUT); no longer HE71.2 (OUTPUT)
- net A63: now also HE78.2 (OUTPUT); no longer HE57.2 (OUTPUT)
- net A68: now also HE43.2 (OUTPUT); no longer HE29.2 (OUTPUT)
- net A71: now also HE29.2 (OUTPUT); no longer HE44.2 (OUTPUT)
- net A72: now also HE44.2 (OUTPUT); no longer HE43.2 (OUTPUT)
- net A77: now also HE60.2 (OUTPUT); no longer HE75.2 (OUTPUT)
- net A78: now also HE75.2 (OUTPUT); no longer HE60.2 (OUTPUT)
