File: HE75.kicad_sch (KiCad schematic)
At the start: 277 parts, among them J1 USB_C_Receptacle_USB2.0_16P, SW1 Esc, SW10 9, SW11 0, SW12 -, SW13 =, SW14 Bksp, SW15 Del, SW16 Tab, SW17 Q, SW18 W, SW19 E, SW2 1, SW20 R, SW21 T, SW22 Y, SW23 U, SW24 I, SW25 O, SW26 P, SW27 [, SW28 ], SW29 \, SW3 2, SW30 Pg Up, SW31 Caps, SW32 A, SW33 S, SW34 D, SW35 F, SW36 G, SW37 H, SW38 J, SW39 K, SW4 3, SW40 L, SW41 ;, SW42 ', SW43 Enter, SW44 Home, SW45 End, SW46 Shift, SW47 Z, SW48 X, SW49 C, SW5 4, SW50 V, SW51 B, SW52 N, SW53 M, SW54 ,, SW55 ., SW56 /, SW57 Shift, SW58 Code, SW59 Up, SW6 5, SW60 Pg Dn, SW61 Fn, SW62 Ctrl, SW63 Win, SW64 Alt, SW65 Space, SW66 Space, SW67 Space, SW68 Space, SW69 Alt, SW7 6, SW70 Win, SW71 Ctrl, SW72 Fn, SW73 Left, SW74 Down, SW75 Right, SW76 Space L2u, SW77 Space C2u, SW78 Space R2u, SW8 7, SW9 8, U1 STM32F303CCT6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

Commit message: Add 6u spacebar stabalizers
Parts:
- added Stab4: MX_stab, PCM_marbastlib-mx:STAB_MX_6u, symbol PCM_marbastlib-mx:MX_stab
Other:
- note added: "2u"
- note removed: "Space C2u"
- note removed: "Space L2u"
- note removed: "Space R2u"
- moved on the sheet: HE77, HE78, Stab2, Stab3, VR77, VR78

Commit message: Adjusting tracks and silkscreens
Parts:
- SW76: value Space L2u -> L2U
- SW77: value Space C2u -> C2U/6U
- SW78: value Space R2u -> R2U
- renumbered RST1 to BOOT0
Other:
- moved on the sheet: Stab4
Changed lines of the file:
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@@
 		(on_board yes)
 		(dnp no)
-		(property "Reference" "RST1"
+		(property "Reference" "BOOT0"
 			(at 63.5 166.37 0)
 			(effects
@@
 			(project "HE75"
 				(path "/92054fa3-5ad0-458e-bd73-acbcf8d11243"
-					(reference "RST1")
+					(reference "BOOT0")
 					(unit 1)
 				)
@@
 			)
 		)
-		(property "Value" "Space L2u"
+		(property "Value" "L2U"
 			(at 321.31 562.61 0)
 			(effects
@@
 	(symbol
 		(lib_id "PCM_marbastlib-mx:MX_stab")
-		(at 401.32 388.62 0)
+		(at 402.59 383.54 0)
 		(unit 1)
 		(exclude_from_sim no)
@@
 		(fields_autoplaced yes)
 		(property "Reference" "Stab4"
-			(at 407.67 387.2229 0)
+			(at 408.94 382.1429 0)
 			(effects
 				(font
@@
 		)
 		(property "Value" "MX_stab"
-			(at 407.67 389.7629 0)
+			(at 408.94 384.6829 0)
 			(effects
 				(font
@@
 		)
 		(property "Footprint" "PCM_marbastlib-mx:STAB_MX_6u"
-			(at 401.32 388.62 0)
+			(at 402.59 383.54 0)
 			(effects
 				(font
@@
 		)
 		(property "Datasheet" ""
-			(at 401.32 388.62 0)
+			(at 402.59 383.54 0)
 			(effects
 				(font
@@
 		)
 		(property "Description" "Cherry MX-style stabilizer"
-			(at 401.32 388.62 0)
+			(at 402.59 383.54 0)
 			(effects
 				(font
@@
 		(fields_autoplaced yes)
 		(property "Reference" "SW77"
-			(at 353.06 558.8 0)
+			(at 356.87 561.3399 0)
 			(effects
 				(font
 					(size 1.27 1.27)
 				)
+				(justify left)
 			)
 		)
-		(property "Value" "Space C2u"
-			(at 353.06 562.61 0)
+		(property "Value" "C2U/6U"
+			(at 356.87 563.8799 0)
 			(effects
 				(font
 					(size 1.27 1.27)
 				)
+				(justify left)
 			)
 		)
@@
 			)
 		)
-		(property "Value" "Space R2u"
+		(property "Value" "R2U"
 			(at 387.35 562.61 0)
 			(effects

Commit message: Fixes for JLCPCB
Parts:
- Stab1: value MX_stab -> Left 2u; footprint PCM_marbastlib-mx:STAB_MX_2u -> Library:STAB_MX_2u; symbol PCM_marbastlib-mx:MX_stab -> Library:MX_stab
- Stab2: value MX_stab -> Center 2u; footprint PCM_marbastlib-mx:STAB_MX_2u -> Library:STAB_MX_2u; symbol PCM_marbastlib-mx:MX_stab -> Library:MX_stab
- Stab3: value MX_stab -> Right 2u; footprint PCM_marbastlib-mx:STAB_MX_2u -> Library:STAB_MX_2u; symbol PCM_marbastlib-mx:MX_stab -> Library:MX_stab
- Stab4: value MX_stab -> Center 6u; footprint PCM_marbastlib-mx:STAB_MX_6u -> Library:STAB_MX_6u; symbol PCM_marbastlib-mx:MX_stab -> Library:MX_stab
- U2: LCSC C2827688 -> C138714
Connections:
- net USB_D+: no longer U2.1 (D1+)
- net USB_D-: no longer U2.5 (D2-)
- no-connect marks 26 -> 30
Changed lines of the file:
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@@
 	)
 	(junction
-		(at 215.9 60.96)
-		(diameter 0)
-		(color 0 0 0 0)
-	)
-	(junction
 		(at 21.59 140.97)
 		(diameter 0)
@@
 	)
 	(junction
-		(at 190.5 66.04)
-		(diameter 0)
-		(color 0 0 0 0)
-	)
-	(junction
 		(at 275.59 271.78)
 		(diameter 0)
@@
 	)
 	(no_connect
+		(at 190.5 60.96)
+	)
+	(no_connect
+		(at 215.9 66.04)
+	)
+	(no_connect
 		(at 64.77 73.66)
 	)
@@
 	)
 	(no_connect
+		(at 215.9 71.12)
+	)
+	(no_connect
 		(at 29.21 88.9)
 	)
@@
 	)
 	(no_connect
+		(at 190.5 55.88)
+	)
+	(no_connect
 		(at 29.21 60.96)
 	)
@@
 	(wire
 		(pts
-			(xy 215.9 60.96) (xy 215.9 66.04)
-		)
-		(stroke
-			(width 0)
-			(type default)
-		)
-	)
-	(wire
-		(pts
 			(xy 443.23 254) (xy 443.23 259.08)
 		)
@@
 	(wire
 		(pts
-			(xy 190.5 60.96) (xy 190.5 66.04)
-		)
-		(stroke
-			(width 0)
-			(type default)
-		)
-	)
-	(wire
-		(pts
 			(xy 339.09 143.51) (xy 344.17 143.51)
 		)
@@
 	)
 	(label "USB_D-"
-		(at 215.9 64.77 0)
+		(at 215.9 60.96 0)
 		(fields_autoplaced yes)
 		(effects
@@
 		)
 	)
-	(label "A47"
-		(at 509.0225 319.3903 0)
-		(fields_autoplaced yes)
-		(effects
-			(font
-				(size 1.27 1.27)
-			)
-			(justify left bottom)
-		)
-	)
 	(label "A57"
 		(at 303.53 143.51 180)
@@
 	)
 	(label "USB_D+"
-		(at 190.5 64.77 180)
+		(at 190.5 66.04 180)
 		(fields_autoplaced yes)
 		(effects
@@
 			)
 		)
-		(property "LCSC" "C2827688"
+		(property "LCSC" "C138714"
 			(at 203.2 63.5 0)
 			(effects
@@
 	)
 	(symbol
-		(lib_id "PCM_marbastlib-mx:MX_stab")
+		(lib_id "Library:MX_stab")
 		(at 402.59 383.54 0)
 		(unit 1)
@@
 			)
 		)
-		(property "Value" "MX_stab"
+		(property "Value" "Center 6u"
 			(at 408.94 384.6829 0)
 			(effects
@@
 			)
 		)
-		(property "Footprint" "PCM_marbastlib-mx:STAB_MX_6u"
+		(property "Footprint" "Library:STAB_MX_6u"
 			(at 402.59 383.54 0)
 			(effects
@@
 	)
 	(symbol
-		(lib_id "PCM_marbastlib-mx:MX_stab")
+		(lib_id "Library:MX_stab")
 		(at 478.79 374.65 0)
 		(unit 1)
@@
 			)
 		)
-		(property "Value" "MX_stab"
+		(property "Value" "Right 2u"
 			(at 485.14 375.7929 0)
 			(effects
@@
 			)
 		)
-		(property "Footprint" "PCM_marbastlib-mx:STAB_MX_2u"
+		(property "Footprint" "Library:STAB_MX_2u"
 			(at 478.79 374.65 0)
 			(effects
@@
 	)
 	(symbol
-		(lib_id "PCM_marbastlib-mx:MX_stab")
+		(lib_id "Library:MX_stab")
 		(at 407.67 373.38 0)
 		(unit 1)
@@
 			)
 		)
-		(property "Value" "MX_stab"
+		(property "Value" "Center 2u"
 			(at 414.02 374.5229 0)
 			(effects
@@
 			)
 		)
-		(property "Footprint" "PCM_marbastlib-mx:STAB_MX_2u"
+		(property "Footprint" "Library:STAB_MX_2u"
 			(at 407.67 373.38 0)
 			(effects
@@
 	)
 	(symbol
-		(lib_id "PCM_marbastlib-mx:MX_stab")
+		(lib_id "Library:MX_stab")
 		(at 336.55 374.65 0)
 		(unit 1)
@@
 			)
 		)
-		(property "Value" "MX_stab"
+		(property "Value" "Left 2u"
 			(at 342.9 375.7929 0)
 			(effects
@@
 			)
 		)
-		(property "Footprint" "PCM_marbastlib-mx:STAB_MX_2u"
+		(property "Footprint" "Library:STAB_MX_2u"
 			(at 336.55 374.65 0)
 			(effects
